File: esp32-c6-xiao-base.kicad_pcb (KiCad board)
At the start: 2 copper layers, 2 parts

Commit message: initial commit with battery connection
Parts:
- added J1: Battery, Connector_PinHeader_2.54mm:PinHeader_1x02_P2.54mm_Horizontal, B.Cu at (176.8, 99.2)
- added R1: 100k, Resistor_SMD:R_0603_1608Metric_Pad0.98x0.95mm_HandSolder, F.Cu at (176.9, 96.2)
- added R2: 100k, Resistor_SMD:R_0603_1608Metric_Pad0.98x0.95mm_HandSolder, F.Cu at (175.2, 96.2)
- added U1: XIAO-ESP32-C6-SMD, Chof747_MCUs:XIAO-ESP32-C6-DIP, F.Cu at (189.4, 100.0)
Routing:
- net BAT-: track 0.00 -> 21.5 mm
- net /BAT_SENSE: track 0.00 -> 20.5 mm
- net BAT+: track 0.00 -> 18.9 mm
Other:
- board outline added: 27.5 x 20 mm
